File: pcb/pcb.kicad_pcb (KiCad board)
At the start: 2 copper layers, 272 x 96 mm, 219 parts, among them J1 Conn_01x12_MountingPin, J2 Conn_01x12_MountingPin

Commit message: initial routing start
Routing:
- net VCC: track 4.02 -> 1339.0 mm, vias 0 -> 65
- net R1: track 0.00 -> 190.3 mm
- net R8: track 0.00 -> 174.0 mm, vias 0 -> 2
- net R7: track 0.00 -> 148.3 mm, vias 0 -> 2
- net R6: track 0.00 -> 132.1 mm
- net R5: track 0.00 -> 127.1 mm
- net R3: track 0.00 -> 122.2 mm
- net R2: track 0.00 -> 122.0 mm
- net R4: track 0.00 -> 93.9 mm
- net (no net): track 0.00 -> 75.9 mm
- net C5: track 0.00 -> 57.4 mm, vias 0 -> 2
- net C2: track 0.00 -> 46.4 mm
- net C6: track 0.00 -> 41.7 mm, vias 0 -> 2
- net Net-(LED59-DOUT): track 0.00 -> 31.3 mm
- net Net-(LED58-DOUT): track 0.00 -> 31.3 mm
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- added copper zone on B.Cu, net GND

Commit message: horizontal routing
Routing:
- net Net-(LED28-DOUT): track 0.00 -> 252.2 mm
- net Net-(LED14-DOUT): track 0.00 -> 248.6 mm
- net Net-(LED41-DOUT): track 0.00 -> 234.7 mm
- net Net-(LED53-DOUT): track 0.00 -> 229.4 mm, vias 0 -> 4
- net VCC: track 1339.0 -> 1260.3 mm, vias 65 -> 0
- net (no net): track 75.9 -> 0.00 mm
- net R4: track 93.9 -> 153.3 mm
- net C5: track 57.4 -> 0.00 mm, vias 2 -> 0
- net C2: track 46.4 -> 0.00 mm
- net C6: track 41.7 -> 0.00 mm, vias 2 -> 0
- net C3: track 28.1 -> 0.00 mm
- net R1: track 190.3 -> 216.6 mm, vias 0 -> 8
- net R8: track 174.0 -> 149.6 mm, vias 2 -> 0
- net RGBIn: track 0.00 -> 21.4 mm
- net R6: track 132.1 -> 153.3 mm
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